File: Documents/B.RobotsJr-KiCad/B.Robots.kicad_sch (KiCad schematic)
At the start: 1 part

Commit message: Add content
Parts:
- added J1: Conn_01x18_Pin, Connector_PinSocket_2.54mm:PinSocket_2x08_P2.54mm_Vertical, symbol Connector:Conn_01x18_Pin
- added J2: Conn_01x04_Pin, symbol Connector:Conn_01x04_Pin
Connections:
- net +5V: now also J1.1 (Pin_1)
- net GND: now also J1.18 (Pin_18)
- net INT2_CAM1: now also J1.13 (Pin_13)
- net RST_CAM1: now also J1.9 (Pin_9)
- net SBL_CAM1: now also J1.10 (Pin_10)
- net SPI1_MISO_CAM1: now also J1.6 (Pin_6)
- net SPI1_MOSI_CAM1: now also J1.7 (Pin_7)
- net SPI1_ON_OF_CAM1: now also J1.8 (Pin_8)
- net SPI1_SCLK_CAM1: now also J1.5 (Pin_5)
- net SPI1_SS_CAM1: now also J1.4 (Pin_4)
- net STLED_CAM1: now also J1.11 (Pin_11)
- net UART1_RX_CAM1: now also J1.2 (Pin_2)
- net UART1_TX_CAM1: now also J1.3 (Pin_3)
- net INT_CAM1 renamed INT1_CAM1
- net INT1_CAM1: now also J1.12 (Pin_12)
- new net USB_5V: J1.14 (Pin_14), J2.4 (Pin_4)
- new net USB_D+: J1.16 (Pin_16), J2.2 (Pin_2)
- new net USB_D-: J1.15 (Pin_15), J2.3 (Pin_3)
- new net USB_GND: J1.17 (Pin_17), J2.1 (Pin_1)
- no-connect marks 8 -> 14
